File: antiThiefSystem/antiThiefSystem.kicad_pcb (KiCad board)
At the start: 4 copper layers, 90 x 60 mm, 26 parts, among them J0 Barrel_Jack, J1 2272-T4, Q0 2SC1815, SW0 SW_SPDT, U1 74LS04, U2 74LS76, U3 74LS08, U4 74LS08, U5 74LS32, U6 NE555D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

Commit message: Finish PCB
Parts:
- moved Q0 79.7 mm to (120.0, 70.0)
- moved R0 76.3 mm to (113.0, 70.0), turned to 180 degrees
- moved BZ0 65.7 mm to (119.0, 84.0), turned to 90 degrees
- moved U6 38.7 mm to (115.0, 93.0)
- moved R3 33.7 mm to (110.0, 98.0), turned to 90 degrees
- moved C1 23.1 mm to (110.0, 104.0), turned to 270 degrees
- moved R2 21.1 mm to (119.0, 105.0)
- moved C0 20.3 mm to (128.0, 98.0), turned to 90 degrees
- moved R1 19.3 mm to (128.0, 104.0), turned to 90 degrees
Connections:
- SW0 pad 1: VCC -> Net-(SW0-Pad1)
- SW0 pad 3: Net-(SW0-Pad3) -> VCC
Routing:
- net GND: track 0.00 -> 295.6 mm, vias 0 -> 6
- net VCC: track 0.00 -> 255.6 mm, vias 0 -> 2
- net /RESET: track 0.00 -> 91.7 mm
- net /CLK: track 0.00 -> 46.3 mm
- net /Q1: track 0.00 -> 36.7 mm
- net /!Q0: track 0.00 -> 21.0 mm
- net Net-(C1-Pad2): track 0.00 -> 19.4 mm
- net Net-(R1-Pad1): track 0.00 -> 18.6 mm
- net Net-(J0-Pad1): track 0.00 -> 18.6 mm
- net Net-(C0-Pad1): track 0.00 -> 17.8 mm
- net /OUT: track 0.00 -> 17.7 mm
- net Net-(BZ0-Pad2): track 0.00 -> 10.9 mm
- net Net-(Q0-Pad1): track 0.00 -> 5.60 mm
- net /LED_B: track 98.4 -> 99.5 mm
- net /LED_A: track 121.8 -> 122.8 mm
